File: KiCad-QTouch-AT42QT2120.kicad_pcb (KiCad board)
At the start: 2 copper layers, 100 x 46 mm, 72 parts, among them J1 Input, J2 Output, U1 AT42QT2120, U2 PCA9635

Commit message: 3D rendering generation with blender
Routing:
- net /OUT2: track 72.7 -> 72.1 mm
Changed lines of the file:
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@@
 	)
 	(via
-		(at 93.75 61)
+		(at 95.531132 61.15)
 		(size 0.6)
 		(drill 0.3)
@@
 	)
 	(via
-		(at 123.147021 75.63862)
+		(at 123.147021 75.65)
 		(size 0.6)
 		(drill 0.3)
@@
 	)
 	(via
-		(at 70 75.75)
+		(at 70 75.65)
 		(size 0.6)
 		(drill 0.3)
@@
 	)
 	(via
-		(at 77.040097 77.864907)
+		(at 77.040097 78.197976)
 		(size 0.6)
 		(drill 0.3)
@@
 	)
 	(via
-		(at 149.25 75.639935)
+		(at 149.25 75.65)
 		(size 0.6)
 		(drill 0.3)
@@
 	)
 	(via
-		(at 88.5 61.75)
+		(at 88.911784 61.15)
 		(size 0.6)
 		(drill 0.3)
@@
 	)
 	(via
-		(at 74 75.5)
+		(at 74 75.65)
 		(size 0.6)
 		(drill 0.3)
@@
 	)
 	(via
-		(at 88.689531 66.433503)
+		(at 88.911784 66.258318)
 		(size 0.6)
 		(drill 0.3)
@@
 	)
 	(via
-		(at 119.531417 74.819132)
+		(at 119.439817 75.004101)
 		(size 0.6)
 		(drill 0.3)
@@
 	)
 	(via
-		(at 140.534526 75.639935)
+		(at 140.534526 75.65)
 		(size 0.6)
 		(drill 0.3)
@@
 	)
 	(via
-		(at 131.819053 75.639935)
+		(at 131.819053 75.65)
 		(size 0.6)
 		(drill 0.3)
@@
 	)
 	(via
-		(at 121.484164 75.645715)
+		(at 121.366686 75.65)
 		(size 0.6)
 		(drill 0.3)
@@
 	)
 	(segment
-		(start 110 56.25)
-		(end 110.5 55.75)
+		(start 98.180664 60.840235)
+		(end 96.405235 60.840235)
 		(width 0.2)
 		(layer "F.Cu")
@@
 	)
 	(segment
-		(start 114.5 55.75)
-		(end 115 56.25)
+		(start 95.75 56.25)
+		(end 110 56.25)
 		(width 0.2)
 		(layer "F.Cu")
@@
 	)
 	(segment
-		(start 95.75 56.25)
-		(end 110 56.25)
+		(start 151.5 57)
+		(end 155.04 60.54)
 		(width 0.2)
 		(layer "F.Cu")
@@
 	)
 	(segment
-		(start 115 56.25)
-		(end 124.25 56.25)
+		(start 94.75 59.185)
+		(end 94.75 57.25)
 		(width 0.2)
 		(layer "F.Cu")
@@
 	)
 	(segment
-		(start 124.25 56.25)
-		(end 125 57)
+		(start 110 56.25)
+		(end 110.5 55.75)
 		(width 0.2)
 		(layer "F.Cu")
@@
 	)
 	(segment
-		(start 151.5 57)
-		(end 155.04 60.54)
+		(start 110.5 55.75)
+		(end 114.5 55.75)
 		(width 0.2)
 		(layer "F.Cu")
@@
 	)
 	(segment
-		(start 110.5 55.75)
-		(end 114.5 55.75)
+		(start 96.405235 60.840235)
+		(end 94.75 59.185)
 		(width 0.2)
 		(layer "F.Cu")
@@
 	)
 	(segment
-		(start 125 57)
-		(end 151.5 57)
+		(start 114.5 55.75)
+		(end 115 56.25)
 		(width 0.2)
 		(layer "F.Cu")
@@
 	)
 	(segment
-		(start 98.180664 60.840235)
-		(end 95.340235 60.840235)
+		(start 98.335664 60.995235)
+		(end 98.180664 60.840235)
 		(width 0.2)
 		(layer "F.Cu")
@@
 	)
 	(segment
-		(start 95.340235 60.840235)
-		(end 94.75 60.25)
+		(start 124.25 56.25)
+		(end 125 57)
 		(width 0.2)
 		(layer "F.Cu")
@@
 	)
 	(segment
-		(start 94.75 60.25)
-		(end 94.75 57.25)
+		(start 155.04 60.54)
+		(end 158 60.54)
 		(width 0.2)
 		(layer "F.Cu")
@@
 	)
 	(segment
-		(start 155.04 60.54)
-		(end 158 60.54)
+		(start 115 56.25)
+		(end 124.25 56.25)
 		(width 0.2)
 		(layer "F.Cu")
@@
 	)
 	(segment
-		(start 98.335664 60.995235)
-		(end 98.180664 60.840235)
+		(start 125 57)
+		(end 151.5 57)
 		(width 0.2)
 		(layer "F.Cu")
@@
 		(polygon
 			(pts
-				(xy 105.340186 73.25) (xy 105.340186 73.25) (xy 105 73.5) (xy 103.5 73.5) (xy 103 74) (xy 103 72.75)
-				(xy 105.340186 72.75)
+				(xy 105.340186 73.25) (xy 105 73.5) (xy 103.5 73.5) (xy 103 74) (xy 103 72.75) (xy 105.340186 72.75)
 			)
 		)
@@
 		(polygon
 			(pts
-				(xy 94.25 62.1547) (xy 94.25 60.1547) (xy 94.75 60.1547) (xy 94.75 62.1547)
+				(xy 96.109466 60.631897) (xy 96.109466 62.156597) (xy 94.244897 62.156597) (xy 94.244897 62.474097)
+				(xy 96.784897 62.474097) (xy 96.784897 62.156597) (xy 96.784897 60.631897)
 			)
 		)
